File: hardware/LM723 voltage regulator.brd (EAGLE design)
At the start: 70 x 80 mm, 41 parts, among them IC1 LM358, J1 CON_TERMINAL_BLOCK_02-5MM, J2 CON_TERMINAL_BLOCK_02-5MM, J3 CON_HEADER_1X03-PTH, Q1 2SA1015, Q2 2N3904, Q3 2N3055, Q4 2SA1015, U1 LM723-EXPAD

Commit message: fix circuit and made 2 panelized board
Parts:
- removed R4: 100K, trosh_devices.eagle.v9:R_5V_EXPAD
- added PAGE1: FRAME_DINA4_L, dp_devices.v6:DP_LOGO
- added R26, R27: 10K, trosh_devices.eagle.v9:R_5V_EXPAD
- R21: value 2.7K -> 5K; device trosh_devices.eagle.v9:R-5_EXPAD -> trosh_devices.eagle.v9:TRIMMER_3362P_EXPAD
- R24, R8: device dp_devices.v6:TRIMMER_3362P -> trosh_devices.eagle.v9:TRIMMER_3362P_EXPAD
- moved R18 7.62 mm to (33.0, 66.0)
- moved IC1 7.62 mm to (36.8, 73.7)
- moved R21 4.02 mm to (25.4, 66.0)
- moved R19 2.54 mm to (45.7, 59.7)
- moved R20 2.54 mm to (38.1, 62.2)
- moved J3 1.27 mm to (3.81, 63.5)
Connections:
- removed net N$5: R4.1, U1.12
- new net N$20: IC1.6, IC1.7
- new net N$21: IC1.5, R26.2, R27.1
- net GND: now also R27.2
- net N$16: now also R21.3
- net VIN: now also R26.1, U1.12; no longer R4.2
Routing:
- net VIN: track 96.9 -> 135.1 mm
- net N$16: track 10.2 -> 23.7 mm
- net N$21: track 0.00 -> 11.7 mm
- net N$18: track 12.0 -> 23.2 mm
- net N$4: track 30.6 -> 23.4 mm
- net N$5: track 5.08 -> 0.00 mm
- net N$20: track 0.00 -> 2.54 mm
- net ADC: track 17.6 -> 16.3 mm
- net !VREG_EN: track 9.94 -> 9.19 mm
Other:
- board text added: "LEADTECH CSPG 10-29-2019"
- board text added: "VREG MODULE V1.0a"
- board text removed: "LEADTECH CSPG 10-23-2019"
- board text removed: "VREG MODULE V1.0"
