File: hardware/leadtech-arduino-CSPG_concept.sch (EAGLE design)
At the start: 41 parts, among them IC3 4050D, J9 CON_HEADER_1X02-PTH, Q1 16Mhz, U1 DS1302, U3 PL2303HX

Commit message: made some rev on dwg and schematic
Other:
- note added: "*GizDuino X 1281 equivalent pins"
- note added: "10"
- note added: "11"
- note added: "12"
- note added: "13"
- note added: "20"
- note added: "21"
- note added: "4"
- note added: "9"
Changed lines of the file:
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@@
 <?xml version="1.0" encoding="utf-8"?>
 <!DOCTYPE eagle SYSTEM "eagle.dtd">
-<eagle version="9.4.2">
+<eagle version="9.1.3">
 <drawing>
 <settings>
@@
 <text x="477.52" y="91.44" size="3.81" layer="94" ratio="12" align="bottom-center">OLED DISPLAY</text>
 <text x="480.06" y="27.94" size="3.81" layer="94" ratio="12" align="bottom-center">PIEZO BEEPER</text>
+<text x="358.14" y="55.88" size="1.778" layer="98" align="center">21</text>
+<text x="358.14" y="58.42" size="1.778" layer="98" align="center">20</text>
+<text x="350.52" y="55.88" size="1.778" layer="98" align="center">4</text>
+<text x="359.664" y="114.046" size="1.778" layer="98" align="center">9</text>
+<text x="359.664" y="109.22" size="1.778" layer="98" align="center">12</text>
+<text x="359.664" y="106.68" size="1.778" layer="98" align="center">11</text>
+<text x="359.664" y="104.14" size="1.778" layer="98" align="center">13</text>
+<text x="359.664" y="101.6" size="1.778" layer="98" align="center">10</text>
+<text x="388.62" y="20.32" size="1.778" layer="98" align="center">*GizDuino X 1281 equivalent pins</text>
 </plain>
 <instances>

Commit message: update files
Parts:
- removed R1: 10K, rcl:R-EU_R0603
Connections:
- removed net N$1: R1.2, SG1.+
- net PIEZO: now also SG1.+; no longer R1.1
Other:
- note added: "2"
Changed lines of the file:
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@@
 <?xml version="1.0" encoding="utf-8"?>
 <!DOCTYPE eagle SYSTEM "eagle.dtd">
-<eagle version="9.1.3">
+<eagle version="9.4.2">
 <drawing>
 <settings>
@@
 <part name="+5V4" library="dp_devices.v6" deviceset="SUPPLY_+5V" device=""/>
 <part name="SG1" library="buzzer" library_urn="urn:adsk.eagle:library:113" deviceset="F/TMB" device="" package3d_urn="urn:adsk.eagle:package:5260/1"/>
-<part name="R1" library="rcl" library_urn="urn:adsk.eagle:library:334" deviceset="R-EU_" device="R0603" package3d_urn="urn:adsk.eagle:package:23555/3" value="10K"/>
 <part name="GND2" library="dp_devices.v6" deviceset="SUPPLY_GND" device=""/>
 <part name="MOD2" library="trosh_devices.eagle.v9" deviceset="OLED_I2C_1.3" device=""/>
@@
 <text x="359.664" y="101.6" size="1.778" layer="98" align="center">10</text>
 <text x="388.62" y="20.32" size="1.778" layer="98" align="center">*GizDuino X 1281 equivalent pins</text>
+<text x="350.52" y="93.98" size="1.778" layer="98" align="center">2</text>
 </plain>
 <instances>
@@
 <attribute name="NAME" x="487.68" y="63.5" size="1.778" layer="95"/>
 <attribute name="VALUE" x="490.22" y="53.34" size="1.778" layer="96" rot="R270"/>
-</instance>
-<instance part="R1" gate="G$1" x="482.6" y="60.96" smashed="yes">
-<attribute name="NAME" x="480.06" y="55.88" size="1.778" layer="95"/>
-<attribute name="VALUE" x="480.06" y="53.34" size="1.778" layer="96"/>
 </instance>
 <instance part="GND2" gate="G$1" x="487.68" y="50.8" smashed="yes"/>
@@
 </segment>
 </net>
-<net name="N$1" class="0">
-<segment>
+<net name="PIEZO" class="0">
+<segment>
+<label x="474.98" y="60.96" size="1.778" layer="95" align="center-right"/>
 <pinref part="SG1" gate="1" pin="+"/>
-<pinref part="R1" gate="G$1" pin="2"/>
-</segment>
-</net>
-<net name="PIEZO" class="0">
-<segment>
-<pinref part="R1" gate="G$1" pin="1"/>
-<wire x1="477.52" y1="60.96" x2="474.98" y2="60.96" width="0.1524" layer="91"/>
-<label x="474.98" y="60.96" size="1.778" layer="95" align="center-right"/>
-</segment>
-<segment>
+<wire x1="474.98" y1="60.96" x2="487.68" y2="60.96" width="0.1524" layer="91"/>
+</segment>
+<segment>

Commit message: small updates
Other:
- note added: "3"
- note added: "PRINTER RX - 3 (PE5)"
- note added: "PRINTER TX - 2 (PE4)"
Changed lines of the file:
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@@
 <text x="388.62" y="20.32" size="1.778" layer="98" align="center">*GizDuino X 1281 equivalent pins</text>
 <text x="350.52" y="93.98" size="1.778" layer="98" align="center">2</text>
+<text x="350.52" y="96.52" size="1.778" layer="98" align="center">3</text>
+<text x="304.8" y="93.98" size="1.778" layer="98" align="center">PRINTER TX - 2 (PE4)</text>
+<text x="304.8" y="96.52" size="1.778" layer="98" align="center">PRINTER RX - 3 (PE5)</text>
 </plain>
 <instances>
@@
 <pinref part="U$1" gate="U" pin="PE5"/>
 <wire x1="340.36" y1="96.52" x2="337.82" y2="96.52" width="0.1524" layer="91"/>
-<label x="337.82" y="96.52" size="1.778" layer="95"/>
-</segment>
-</net>
+<label x="337.82" y="96.52" size="1.778" layer="95" align="center-right"/>
+</segment>
+</net>

Commit message: add gizduino pins on schematic, add bug comment on value of month on vendor firmware, add time sketches
Other:
- note added: "5"
- note added: "6"
- note added: "7"
Changed lines of the file:
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@@
 <text x="304.8" y="93.98" size="1.778" layer="98" align="center">PRINTER TX - 2 (PE4)</text>
 <text x="304.8" y="96.52" size="1.778" layer="98" align="center">PRINTER RX - 3 (PE5)</text>
+<text x="359.664" y="119.126" size="1.778" layer="98" align="center">7</text>
+<text x="359.664" y="116.586" size="1.778" layer="98" align="center">6</text>
+<text x="350.52" y="91.44" size="1.778" layer="98" align="center">5</text>
 </plain>
 <instances>

Commit message: 1
Parts:
- removed MOD1: RFIO-RC522, trosh_devices.eagle.v9:RFIO-RC522
- removed MOD2: OLED_I2C_1.3, trosh_devices.eagle.v9:OLED_I2C_1.3
- added J1: CON_HEADER_1X08-PTH, dp_devices.v6:CON_HEADER_1X08-PTH
- added J2: CON_HEADER_1X04, dp_devices.v6:CON_HEADER_1X04
- added J3: CON_HEADER_1X03-PTH, dp_devices.v6:CON_HEADER_1X03-PTH
Connections:
- new net N$1: J3.3
- new net N$2: J3.2
- net +3V3: now also J1.8; no longer MOD1.+3V3
- net +5V: now also J2.1, LED2.A; no longer MOD2.VCC
- net DISPLAY_I2C_CLOCK: now also J2.3; no longer MOD2.SCL
- net DISPLAY_I2C_DATA: now also J2.4; no longer MOD2.SDA
- net GND: now also J1.6, J2.2, J3.1; no longer MOD1.GND, MOD2.GND
- net RFID_CLOCK_3V: now also J1.2; no longer MOD1.SCK
- net RFID_DATA_3V: now also J1.1; no longer MOD1.SDA
- net RFID_MISO: now also J1.4; no longer MOD1.MISO
- net RFID_MOSI_3V: now also J1.3; no longer MOD1.MOSI
- net RFID_RESET_3V: now also J1.7; no longer MOD1.RST

Commit message: edit CSPG arduino hardware
Parts:
- added R1: 10K, rcl:R-EU_R0603
Connections:
- new net N$3: R1.1, U$1.!RST
- net +5V: now also R1.2
Changed lines of the file:
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@@
 <part name="J2" library="dp_devices.v6" deviceset="CON_HEADER_1X04" device=""/>
 <part name="J3" library="dp_devices.v6" deviceset="CON_HEADER_1X03" device="-PTH"/>
+<part name="R1" library="rcl" library_urn="urn:adsk.eagle:library:334" deviceset="R-EU_" device="R0603" package3d_urn="urn:adsk.eagle:package:23555/3" value="10K"/>
+<part name="+5V1" library="dp_devices.v6" deviceset="SUPPLY_+5V" device=""/>
 </parts>
 <sheets>
@@
 <instance part="J2" gate="J" x="487.68" y="134.62"/>
 <instance part="J3" gate="J" x="284.48" y="83.82" rot="MR0"/>
+<instance part="R1" gate="G$1" x="337.82" y="149.86" smashed="yes" rot="R90">
+<attribute name="NAME" x="340.36" y="149.86" size="1.778" layer="95"/>
+<attribute name="VALUE" x="340.36" y="147.32" size="1.778" layer="96"/>
+</instance>
+<instance part="+5V1" gate="SUPPLY" x="337.82" y="157.48" smashed="yes"/>
 </instances>
 <busses>
@@
 <wire x1="487.68" y1="137.16" x2="485.14" y2="137.16" width="0.1524" layer="91"/>
 <label x="485.14" y="137.16" size="1.778" layer="95" align="center-right"/>
+</segment>
+<segment>
+<pinref part="R1" gate="G$1" pin="2"/>
+<pinref part="+5V1" gate="SUPPLY" pin="+5V"/>
+<wire x1="337.82" y1="154.94" x2="337.82" y2="157.48" width="0.1524" layer="91"/>
+<label x="337.82" y="160.02" size="1.778" layer="95"/>
 </segment>
 </net>
@@
 </segment>
 </net>
+<net name="N$3" class="0">
+<segment>
+<pinref part="U$1" gate="U" pin="!RST"/>
+<wire x1="340.36" y1="142.24" x2="337.82" y2="142.24" width="0.1524" layer="91"/>
+<pinref part="R1" gate="G$1" pin="1"/>
+<wire x1="337.82" y1="142.24" x2="337.82" y2="144.78" width="0.1524" layer="91"/>
+</segment>
+</net>

Commit message: worked on schematic
Parts:
- added IC1: OP-AMP, SparkFun-IC-Amplifiers:OPAMP-DUALU
- added Q2: (no value), dp_devices.v6:TRANSISTOR_FET_TSM2301CX
- added R11: 330R, dp_devices.v6:RESISTOR-0603
- added VREG2: 3.3V, dp_devices.v6:VREG_3PINS-SOT-223
Connections:
- new net N$4: IC1G1.OUT, Q2.G
- net +3V3: now also IC1G1.-IN, VREG2.VOUT
- net +5V: now also IC1G3.P$V+, Q2.S, VREG2.VIN
- net GND: now also IC1G3.P$V-, VREG2.GND
- net VUSB: now also Q2.D

Commit message: 1
Parts:
- added C1: 10uF, dp_devices.v6:CAPACITOR_POL-CASE_B
- added R12: 10K, dp_devices.v6:RESISTOR-0603
- R11: value 330R -> 10K
Connections:
- removed net N$20: C8.+, D1.C, VREG1.VIN
- new net N$5: IC1G1.+IN, R11.1, R12.2
- new net VIN: C8.+, D1.C, R11.2, VREG1.VIN
- net +3V3: now also C1.+
- net GND: now also C1.-, R12.1
Other:
- moved on the sheet: R11
Changed lines of the file:
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@@
 <?xml version="1.0" encoding="utf-8"?>
 <!DOCTYPE eagle SYSTEM "eagle.dtd">
-<eagle version="9.1.3">
+<eagle version="9.4.2">
 <drawing>
 <settings>
@@
 <part name="Q2" library="dp_devices.v6" deviceset="TRANSISTOR_FET_TSM2301CX" device=""/>
 <part name="+5V3" library="dp_devices.v6" deviceset="SUPPLY_+5V" device=""/>
-<part name="R11" library="dp_devices.v6" deviceset="RESISTOR" device="-0603" value="330R"/>
+<part name="R11" library="dp_devices.v6" deviceset="RESISTOR" device="-0603" value="10K"/>
 <part name="VREG2" library="dp_devices.v6" deviceset="VREG_3PINS" device="-SOT-223" value="3.3V"/>
 <part name="GND1" library="dp_devices.v6" deviceset="SUPPLY_GND" device=""/>
@@
 <part name="+5V19" library="dp_devices.v6" deviceset="SUPPLY_+5V" device=""/>
 <part name="+5V20" library="dp_devices.v6" deviceset="SUPPLY_+5V" device=""/>
+<part name="C1" library="dp_devices.v6" deviceset="CAPACITOR_POL" device="-CASE_B" value="10uF"/>
+<part name="GND4" library="dp_devices.v6" deviceset="SUPPLY_GND" device=""/>
+<part name="R12" library="dp_devices.v6" deviceset="RESISTOR" device="-0603" value="10K"/>
+<part name="GND5" library="dp_devices.v6" deviceset="SUPPLY_GND" device=""/>
+<part name="+5V21" library="dp_devices.v6" deviceset="SUPPLY_+5V" device=""/>
+<part name="+5V22" library="dp_devices.v6" deviceset="SUPPLY_+5V" device=""/>
 </parts>
 <sheets>
@@
 </instance>
 <instance part="C8" gate="C" x="48.26" y="154.94" smashed="yes">
-<attribute name="NAME" x="48.26" y="162.56" size="1.778" layer="95"/>
-<attribute name="VALUE" x="48.26" y="160.02" size="1.778" layer="96"/>
+<attribute name="NAME" x="50.8" y="152.4" size="1.778" layer="95"/>
+<attribute name="VALUE" x="50.8" y="149.86" size="1.778" layer="96"/>
 </instance>
 <instance part="VREG1" gate="VREG" x="66.04" y="157.48" smashed="yes">
@@
 </instance>
 <instance part="+5V17" gate="SUPPLY" x="464.82" y="147.32" smashed="yes"/>
-<instance part="J1" gate="J" x="233.68" y="142.24"/>
-<instance part="J2" gate="J" x="487.68" y="134.62"/>
-<instance part="J3" gate="J" x="284.48" y="83.82" rot="MR0"/>
+<instance part="J1" gate="J" x="233.68" y="142.24" smashed="yes">
+<attribute name="NAME" x="232.41" y="153.035" size="1.778" layer="95"/>
+</instance>
+<instance part="J2" gate="J" x="487.68" y="134.62" smashed="yes">
+<attribute name="NAME" x="486.41" y="140.97" size="1.778" layer="95"/>
+</instance>
+<instance part="J3" gate="J" x="284.48" y="83.82" smashed="yes" rot="MR0">
+<attribute name="NAME" x="285.75" y="90.17" size="1.778" layer="95" rot="MR0"/>
+</instance>
 <instance part="R1" gate="G$1" x="337.82" y="149.86" smashed="yes" rot="R90">
 <attribute name="NAME" x="340.36" y="149.86" size="1.778" layer="95"/>
@@
 </instance>
 <instance part="+5V1" gate="SUPPLY" x="337.82" y="157.48" smashed="yes"/>
-<instance part="IC1" gate="G1" x="185.42" y="226.06"/>
-<instance part="Q2" gate="Q" x="208.28" y="231.14" rot="R90"/>
+<instance part="IC1" gate="G1" x="185.42" y="226.06" smashed="yes">
+<attribute name="NAME" x="180.34" y="231.902" size="1.778" layer="95" font="vector"/>
+<attribute name="VALUE" x="180.34" y="218.44" size="1.778" layer="95" font="vector"/>
+</instance>
+<instance part="Q2" gate="Q" x="208.28" y="231.14" smashed="yes" rot="R90">
+<attribute name="VALUE" x="208.28" y="219.71" size="1.778" layer="96" rot="R90"/>
+<attribute name="NAME" x="205.74" y="219.71" size="1.778" layer="95" rot="R90"/>
+</instance>
 <instance part="+5V3" gate="SUPPLY" x="200.66" y="238.76" smashed="yes"/>
-<instance part="R11" gate="R" x="154.94" y="238.76" smashed="yes" rot="R90">
-<attribute name="NAME" x="149.86" y="236.22" size="1.778" layer="95" font="vector" rot="R90"/>
-<attribute name="VALUE" x="152.4" y="236.22" size="1.778" layer="96" font="vector" rot="R90"/>
-</instance>
-<instance part="VREG2" gate="VREG" x="238.76" y="233.68"/>
+<instance part="R11" gate="R" x="165.1" y="231.14" smashed="yes" rot="R90">
+<attribute name="NAME" x="160.02" y="228.6" size="1.778" layer="95" font="vector" rot="R90"/>
+<attribute name="VALUE" x="162.56" y="228.6" size="1.778" layer="96" font="vector" rot="R90"/>
+</instance>
+<instance part="VREG2" gate="VREG" x="238.76" y="233.68" smashed="yes">
+<attribute name="NAME" x="231.14" y="239.522" size="1.778" layer="95"/>
+<attribute name="VALUE" x="231.14" y="237.236" size="1.778" layer="96"/>
+</instance>
 <instance part="GND1" gate="G$1" x="238.76" y="223.52" smashed="yes"/>
-<instance part="IC1" gate="G3" x="182.88" y="254"/>
-<instance part="IC1" gate="G2" x="162.56" y="266.7"/>
+<instance part="IC1" gate="G3" x="182.88" y="254" smashed="yes">
+<attribute name="NAME" x="179.578" y="248.92" size="1.778" layer="95" font="vector" rot="R90"/>
+<attribute name="VALUE" x="187.96" y="248.92" size="1.778" layer="95" font="vector" rot="R90"/>
+</instance>
+<instance part="IC1" gate="G2" x="162.56" y="266.7" smashed="yes">
+<attribute name="NAME" x="157.48" y="272.542" size="1.778" layer="95" font="vector"/>
+<attribute name="VALUE" x="157.48" y="259.08" size="1.778" layer="95" font="vector"/>
+</instance>
 <instance part="GND3" gate="G$1" x="182.88" y="243.84" smashed="yes"/>
 <instance part="+5V5" gate="SUPPLY" x="182.88" y="264.16" smashed="yes"/>
@@
 <instance part="+5V19" gate="SUPPLY" x="254" y="238.76" smashed="yes"/>
 <instance part="+5V20" gate="SUPPLY" x="172.72" y="231.14" smashed="yes"/>
+<instance part="C1" gate="C" x="254" y="231.14" smashed="yes">
+<attribute name="NAME" x="256.54" y="231.14" size="1.778" layer="95"/>
+<attribute name="VALUE" x="256.54" y="228.6" size="1.778" layer="96"/>
+</instance>
+<instance part="GND4" gate="G$1" x="254" y="223.52" smashed="yes"/>
+<instance part="R12" gate="R" x="165.1" y="215.9" smashed="yes" rot="R90">
+<attribute name="NAME" x="160.02" y="213.36" size="1.778" layer="95" font="vector" rot="R90"/>
+<attribute name="VALUE" x="162.56" y="213.36" size="1.778" layer="96" font="vector" rot="R90"/>
+</instance>
+<instance part="GND5" gate="G$1" x="165.1" y="208.28" smashed="yes"/>
+<instance part="+5V21" gate="SUPPLY" x="48.26" y="162.56" smashed="yes"/>
+<instance part="+5V22" gate="SUPPLY" x="165.1" y="238.76" smashed="yes"/>
 </instances>
 <busses>
@@
 <pinref part="IC1" gate="G3" pin="P$V-"/>
 <pinref part="GND3" gate="G$1" pin="GND"/>
+</segment>
+<segment>
+<pinref part="C1" gate="C" pin="-"/>
+<pinref part="GND4" gate="G$1" pin="GND"/>
+</segment>
+<segment>
+<pinref part="R12" gate="R" pin="1"/>
+<pinref part="GND5" gate="G$1" pin="GND"/>
 </segment>
 </net>
@@
 </segment>
 </net>
-<net name="N$20" class="0">
-<segment>
-<pinref part="D1" gate="1" pin="C"/>
-<pinref part="C8" gate="C" pin="+"/>
-<wire x1="43.18" y1="157.48" x2="48.26" y2="157.48" width="0.1524" layer="91"/>
-<pinref part="VREG1" gate="VREG" pin="VIN"/>
-<wire x1="48.26" y1="157.48" x2="55.88" y2="157.48" width="0.1524" layer="91"/>
-<junction x="48.26" y="157.48"/>
-</segment>
-</net>
 <net name="N$21" class="0">
 <segment>
@@
 <wire x1="254" y1="236.22" x2="254" y2="238.76" width="0.1524" layer="91"/>
 <label x="254" y="241.3" size="1.778" layer="95"/>
+<pinref part="C1" gate="C" pin="+"/>
+<junction x="254" y="233.68"/>
 </segment>
 <segment>
@@
 </segment>
 </net>
+<net name="N$5" class="0">
+<segment>
+<pinref part="IC1" gate="G1" pin="+IN"/>
+<wire x1="177.8" y1="223.52" x2="165.1" y2="223.52" width="0.1524" layer="91"/>
+<pinref part="R11" gate="R" pin="1"/>
+<wire x1="165.1" y1="223.52" x2="165.1" y2="226.06" width="0.1524" layer="91"/>
+<pinref part="R12" gate="R" pin="2"/>
+<wire x1="165.1" y1="220.98" x2="165.1" y2="223.52" width="0.1524" layer="91"/>
+<junction x="165.1" y="223.52"/>
+</segment>
+</net>
+<net name="VIN" class="0">
+<segment>
+<pinref part="D1" gate="1" pin="C"/>
+<pinref part="C8" gate="C" pin="+"/>
+<wire x1="43.18" y1="157.48" x2="48.26" y2="157.48" width="0.1524" layer="91"/>
+<pinref part="VREG1" gate="VREG" pin="VIN"/>
+<wire x1="48.26" y1="157.48" x2="55.88" y2="157.48" width="0.1524" layer="91"/>
+<junction x="48.26" y="157.48"/>
+<pinref part="+5V21" gate="SUPPLY" pin="+5V"/>
+<wire x1="48.26" y1="157.48" x2="48.26" y2="162.56" width="0.1524" layer="91"/>
+<label x="48.26" y="165.1" size="1.778" layer="95"/>
+</segment>
+<segment>
+<pinref part="R11" gate="R" pin="2"/>
+<wire x1="165.1" y1="236.22" x2="165.1" y2="238.76" width="0.1524" layer="91"/>
+<pinref part="+5V22" gate="SUPPLY" pin="+5V"/>
+<label x="165.1" y="241.3" size="1.778" layer="95"/>
+</segment>
+</net>
