File: hardware/leadtech-arduino-CSPG_concept.sch (EAGLE design)
At the start: 63 parts, among them IC1 OP-AMP, IC3 4050D, J1 CON_HEADER_1X08-PTH, J3 CON_HX42003_2, J5 CON_HEADER_1X02-PTH, J6 2510-4AGW, J9 CON_HEADER_1X02-PTH, Q1 16Mhz, U1 DS1302, U2 VREG-78M05, U3 PL2303HX, U4 MP1584EN_MODULE, U5 RT9163-3.3V, U6 ATMEGA1281, U7 AZ1117CH2-3.3TRG1

Commit message: done routing, add bom
Parts:
- removed J6: 2510-4AGW, trosh_devices.eagle.v9:CON_KF2510-4AGW-2
- removed Q2: (no value), dp_devices.v6:TRANSISTOR_FET_TSM2301CX
- added J4: CON_KF2510-2AGW, trosh_devices.eagle.v9:CON_KF2510-2AGW
- added X1: 16Mhz, special:XTAL/S
- C14, C15: value 0.1uF -> 22pF; device rcl:C-EUC0603 -> dp_devices.v6:CAPACITOR_NPOL-0805
- C16: value 0.1uF -> 10uF; device rcl:C-EUC0603 -> dp_devices.v6:CAPACITOR_POL-CASE_B
- C18: value 10uF -> 0.1uF; device dp_devices.v6:CAPACITOR_POL-CASE_B -> rcl:C-EUC0603
- C2: value 22pF -> 10uF; device dp_devices.v6:CAPACITOR_NPOL-0805 -> rcl:C-EUC0805
- C3: value 22pF -> 100uF; device dp_devices.v6:CAPACITOR_NPOL-0805 -> dp_devices.v6:CAPACITOR_POL-CASE_B
- C5: value 10uF -> 0.1uF; device rcl:C-EUC0805 -> rcl:C-EUC0603
- C7: value 0.1uF -> 100uF; device rcl:C-EUC0603 -> dp_devices.v6:CAPACITOR_POL-CASE_B
- C8, C9: value 100uF -> 0.1uF; device dp_devices.v6:CAPACITOR_POL-CASE_B -> rcl:C-EUC0603
- J1: value CON_HEADER_1X08-PTH -> CON_HX42003_2; device dp_devices.v6:CON_HEADER_1X08-PTH -> trosh_devices.eagle.v9:CON_HX42003_2
- J3: value CON_HX42003_2 -> 2510-4AGW; device trosh_devices.eagle.v9:CON_HX42003_2 -> trosh_devices.eagle.v9:CON_KF2510-4AGW-2
- J5: value CON_HEADER_1X02-PTH -> CON_HEADER_1X08-PTH; device dp_devices.v6:CON_HEADER_1X02-PTH -> dp_devices.v6:CON_HEADER_1X08-PTH
- Q1: value 16Mhz -> (none); device special:XTAL/S -> dp_devices.v6:TRANSISTOR_FET_TSM2301CX
- R1: value 10K -> 1.5K; device rcl:R-EU_R0603 -> dp_devices.v6:RESISTOR-0603
- R10, R5: device rcl:R-EU_R0603 -> dp_devices.v6:RESISTOR-0603
- R11, R12, R13, R14: device dp_devices.v6:RESISTOR-0603 -> rcl:R-EU_R0603
- R15: value 100R -> 10K; device rcl:R-EU_R0603 -> dp_devices.v6:RESISTOR-0603
- R16: value 10K -> 100R; device dp_devices.v6:RESISTOR-0603 -> rcl:R-EU_R0603
- R2: value 10K -> 27R; device rcl:R-EU_R0603 -> dp_devices.v6:RESISTOR-0603
- R4: value 27R -> 330R
- R6: value 1.5K -> 10K
- R9: value 330R -> 10K
- U1: value DS1302 -> MP1584EN_MODULE; device trosh_devices.eagle.v9:DS1302 -> trosh_devices.eagle.v9:MP1584EN_MODULE
- U4: value MP1584EN_MODULE -> RT9163-3.3V; device trosh_devices.eagle.v9:MP1584EN_MODULE -> trosh_devices.eagle.v9:VREG-RT9163
- U5: value RT9163-3.3V -> DS1302; device trosh_devices.eagle.v9:VREG-RT9163 -> trosh_devices.eagle.v9:DS1302
- renumbered IC1 to U8, IC3 to U9, J9 to J2, LED2 to LED1, MOD1 to U10, XTAL1 to X2
Connections:
- net +3V3: now also C7.+, C8.2, J5.8, U4.VOUT; no longer C1.+, C15.2, J1.8, R16.2, R17.2, R19.1, R20.1, U5.VOUT
- net +3V3_ESP: now also C18.2, R15.2, R17.2, R18.1, R19.1; no longer C14.2
- net +5V: now also C16.+, C3.+, C9.2, J3.4, Q1.S, R11.2, R12.2, R14.2, R9.2, U4.VIN, U5.VCC2; no longer C16.2, C18.+, C9.+, J6.4, Q2.S, R1.2, R10.2, R2.2, R5.2, U1.VCC2, U5.VIN
- net DISPLAY_I2C_CLOCK: now also J3.2, R14.1; no longer J6.2, R2.1
- net DISPLAY_I2C_DATA: now also J3.1, R13.1; no longer J6.1, R10.1
- net GND: now also C14.2, C16.-, C18.1, C3.-, C4.1, C6.2, C7.-, C8.1, C9.1, J1.2, J3.3, J4.2, J5.6, L1.1, R10.1, R20.1, R4.2, R6.1, U1.VIN-, U1.VOUT-, U4.GND; no longer C14.1, C16.1, C18.-, C3.1, C4.2, C6.1, C7.2, C8.-, C9.-, J1.6, J3.2, J5.2, J6.3, L2.1, R12.1, R14.1, R18.1, R9.2, U1.GND, U4.VIN-, U4.VOUT-
- net N$1: now also R17.1; no longer R16.1
- net N$10: now also C14.1, X1.1; no longer C2.1, Q1.1
- net N$11: now also R2.1; no longer R3.1
- net N$12: now also R1.1, R3.1; no longer R4.1, R6.1
- net N$13: now also R2.2; no longer R3.2
- net N$14: now also R3.2; no longer R4.2
- net N$15: now also L2.2; no longer L1.2
- net N$16: now also L1.2; no longer L2.2
- net N$19: now also U1.VOUT+; no longer U4.VOUT+
- net N$2: now also R15.1; no longer R17.1
- net N$20: now also R16.2; no longer R15.2
- net N$21: now also R4.1; no longer R9.1
- net N$22: now also U5.X2; no longer U1.X2
- net N$23: now also U5.X1; no longer U1.X1
- net N$24: now also U5.VCC1; no longer U1.VCC1
- net N$25: now also R20.2; no longer R18.2
- net N$27: now also R18.2; no longer R20.2
- net N$3: now also R12.1; no longer R1.1
- net N$4: now also Q1.G; no longer Q2.G
- net N$5: now also R5.1, R6.2; no longer R11.1, R12.2
- net N$7: now also J1.1, U1.VIN+; no longer J3.1, U4.VIN+
- net N$8: now also C15.2, X1.2; no longer C3.2, Q1.2
- net N$9: now also R10.2, R9.1; no longer R13.1, R14.2
- net PIEZO: now also R16.1; no longer R15.1
- net RFID_CLOCK_3V: now also J5.2; no longer J1.2
- net RFID_DATA_3V: now also J5.1; no longer J1.1
- net RFID_MISO: now also J5.4; no longer J1.4
- net RFID_MOSI_3V: now also J5.3; no longer J1.3
- net RFID_RESET_3V: now also J5.7; no longer J1.7
- net RTC_CLOCK: now also U5.SCLK; no longer U1.SCLK
- net RTC_DATA: now also U5.I/O; no longer U1.I/O
- net RTC_EN: now also U5.CE; no longer U1.CE
- net SW1: now also J4.1, R11.1; no longer J5.1, R5.1
- net VIN: now also C1.+, R5.2; no longer C8.+, R11.2
- net VO33: now also C5.1, C6.1, R1.2; no longer C4.1, C7.1, R6.2
- net VUSB: now also C2.1, C4.2, L2.1, Q1.D; no longer C5.1, C6.2, L1.1, Q2.D
Other:
- note added: "3.3V Only"
- note added: "Dedicated VREG needs >500mA"
- moved on the sheet: C1, C4, C5, C6, L1, L2, R17, R18, R20, R3, R4, R6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

Commit message: making bom
Parts:
- C1, C3, C7: value 100uF -> 100uF 16V; device dp_devices.v6:CAPACITOR_POL-CASE_B -> trosh_devices.eagle.v9:CAPACITOR-POLCASE_C
- C14, C15: device dp_devices.v6:CAPACITOR_NPOL-0805 -> rcl:C-EUC0603
- C16, C17: value 10uF -> 10uF 16V
- C2: device rcl:C-EUC0805 -> rcl:C-EUC0603
Connections:
- net GND: now also C14.1, C2.1, U9E.I; no longer C14.2, C2.2
- net N$10: now also C14.2; no longer C14.1
- net VUSB: now also C2.2; no longer C2.1
Other:
- moved on the sheet: C2
