File: hardware/LM723 voltage regulator.v1.0a.brd (EAGLE design)
At the start: 70 x 80 mm, 43 parts, among them IC1 LM358, J1 CON_TERMINAL_BLOCK_02-5MM, J2 CON_TERMINAL_BLOCK_02-5MM, J3 CON_HEADER_1X03-PTH, Q1 2SA1015, Q2 2N3904, Q3 2N3055, Q4 2SA1015, U1 LM723-EXPAD

Commit message: revision on main board
Parts:
- R8: value 5K -> 10K
Changed lines of the file:
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@@
 <?xml version="1.0" encoding="utf-8"?>
 <!DOCTYPE eagle SYSTEM "eagle.dtd">
-<eagle version="9.4.2">
+<eagle version="9.1.3">
 <drawing>
 <settings>
@@
 <attribute name="VALUE" x="29.8958" y="5.334" size="1.27" layer="27" ratio="10" rot="R90"/>
 </element>
-<element name="R8" library="trosh_devices.eagle.v9" package="TRIMMER_3362P_EXPAD" value="5K" x="41.91" y="7.62" smashed="yes" rot="R180">
+<element name="R8" library="trosh_devices.eagle.v9" package="TRIMMER_3362P_EXPAD" value="10K" x="41.91" y="7.62" smashed="yes" rot="R180">
 <attribute name="NAME" x="45.085" y="3.81" size="1.27" layer="25" ratio="10" rot="R180"/>
 <attribute name="VALUE" x="45.085" y="13.0175" size="1.27" layer="27" ratio="10" rot="R180"/>
