File: hardware/LM723 voltage regulator.v1.0a.sch (EAGLE design)
At the start: 43 parts, among them IC1 LM358, J1 CON_TERMINAL_BLOCK_02-5MM, J2 CON_TERMINAL_BLOCK_02-5MM, J3 CON_HEADER_1X03-PTH, Q1 2SA1015, Q2 2N3904, Q3 2N3055, Q4 2SA1015, U1 LM723-EXPAD

Commit message: revision on main board
Parts:
- R8: value 5K -> 10K
Changed lines of the file:
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@@
 <?xml version="1.0" encoding="utf-8"?>
 <!DOCTYPE eagle SYSTEM "eagle.dtd">
-<eagle version="9.4.2">
+<eagle version="9.1.3">
 <drawing>
 <settings>
@@
 <part name="R7" library="trosh_devices.eagle.v9" deviceset="RESISTOR" device="-V" value="100K"/>
 <part name="GND4" library="dp_devices.v6" deviceset="SUPPLY_GND" device=""/>
-<part name="R8" library="trosh_devices.eagle.v9" deviceset="TRIMMER" device="-3362P_EXPAD" value="5K"/>
+<part name="R8" library="trosh_devices.eagle.v9" deviceset="TRIMMER" device="-3362P_EXPAD" value="10K"/>
 <part name="R9" library="trosh_devices.eagle.v9" deviceset="RESISTOR" device="-V" value="3.3K"/>
 <part name="R10" library="rcl" library_urn="urn:adsk.eagle:library:334" deviceset="R-EU_" device="0207/12" package3d_urn="urn:adsk.eagle:package:23489/1" value="10K"/>
