File: hardware/leadtech-arduino-CSPG_concept.brd (EAGLE design)
At the start: 80 x 61 mm, 63 parts, among them J1 CON_HX42003_2, J2 CON_HEADER_1X02-PTH, J3 2510-4AGW, J4 CON_KF2510-2AGW, J5 CON_HEADER_1X08-PTH, U1 MP1584EN_MODULE, U10 ESP8266-07, U2 VREG-78M05, U3 PL2303HX, U4 RT9163-3.3V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

Commit message: making bom
Parts:
- C1, C3, C7: value 100uF -> 100uF 16V; device dp_devices.v6:CASE_B -> trosh_devices.eagle.v9:CASE_C
- C14, C15: device dp_devices.v6:C805 -> rcl:C0603
- C16, C17: value 10uF -> 10uF 16V
- C2: device rcl:C0805 -> rcl:C0603
- turned C14 to 270 degrees
- turned C2 to 90 degrees
Connections:
- net GND: now also C14.1, C2.1, U9.11; no longer C14.2, C2.2
- net N$10: now also C14.2; no longer C14.1
- net VUSB: now also C2.2; no longer C2.1
Routing:
- net RFID_MOSI_3V: track 16.0 -> 12.7 mm
- net RFID_CLOCK_3V: track 19.2 -> 16.0 mm
- net RFID_DATA_3V: track 22.4 -> 19.6 mm
- net N$28: track 47.9 -> 47.1 mm
- net VIN: track 48.9 -> 48.3 mm
Other:
- board text added: "POWER"

Commit message: finish routing main board and bom
Parts:
- removed R1: 1.5K, dp_devices.v6:R603
- removed R2, R3: 27R, dp_devices.v6:R603
- U2: value VREG-78M05 -> L7805; device trosh_devices.eagle.v9:DPAK-3 -> trosh_devices.eagle.v9:DPAK
- U3: value PL2303HX -> PL2303TA
- USB1: value USB-F-MINI-B -> CON-USB-F-MICRO-B-2; device dp_devices.v6:CONN_USB_MINI-B -> dp_devices.v6:CON_USB_MICRO-B-2-SD-47589-001
- moved C10 18.5 mm to (61.0, 1.91), turned to 0 degrees
- moved C6 15.5 mm to (67.9, 19.7), turned to 90 degrees
- moved C5 13.2 mm to (61.6, 6.99), turned to 0 degrees
- moved D1 9.69 mm to (61.6, 52.7), turned to 0 degrees
- moved U3 5.90 mm to (62.9, 12.7), turned to 0 degrees
- moved R7 5.85 mm to (54.6, 12.0)
- moved C2 5.68 mm to (73.7, 8.89), turned to 180 degrees
- moved X2 5.15 mm to (59.7, 4.45)
- moved USB1 4.22 mm to (78.9, 14.0)
- moved U5 4.07 mm to (51.4, 4.45), turned to 90 degrees
- moved R8 4.02 mm to (54.6, 13.9)
- moved C4 3.15 mm to (54.6, 15.9)
- moved L1 2.62 mm to (71.1, 17.8)
- moved L2 2.54 mm to (71.1, 10.8)
- moved U2 1.91 mm to (62.2, 47.6)
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Connections:
- removed net N$13: R2.2, U3.P16
- removed net N$14: R3.2, U3.P15
- net N$11: now also U3.P16, USB1.P2; no longer R2.1, USB1.D-
- net N$12: now also U3.P15, USB1.P3; no longer R1.1, R3.1, USB1.D+
- net N$15: now also USB1.P1; no longer USB1.VUSB
- net N$16: now also USB1.P5; no longer USB1.GND
- net VO33: no longer R1.2
Routing:
- net +5V: track 274.0 -> 210.2 mm, vias 11 -> 14
- net N$19: track 26.5 -> 0.00 mm
- net VO33: track 32.6 -> 20.6 mm, vias 0 -> 2
- net N$14: track 11.9 -> 0.00 mm
- net VUSB: track 33.3 -> 21.5 mm, vias 3 -> 5
- net N$13: track 8.27 -> 0.00 mm
- net RTC_CLOCK: track 40.9 -> 49.1 mm
- net N$24: track 4.11 -> 12.1 mm
- net N$18: track 2.37 -> 8.23 mm
- net UART_RX: track 23.4 -> 29.1 mm
- net VIN: track 48.3 -> 42.6 mm
- net RTC_DATA: track 40.1 -> 45.6 mm
- net N$11: track 5.76 -> 11.2 mm
- net N$23: track 6.99 -> 3.64 mm
- net N$12: track 7.24 -> 10.1 mm
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- added copper zone on layer 1, net +5V
- added copper zone on layer 16, net +5V
- added copper zone on layer 1, net N$19
- added copper zone on layer 1, net VIN
- added copper zone on layer 1, net VUSB
- added copper zone on layer 16, net VUSB

Commit message: revision on main board
Parts:
- added F1: 6V/0.75A, SparkFun-Fuses:1206
- added J6: (no value), trosh_devices.eagle.v9:KF2510-3A
- moved C2 5.88 mm to (68.7, 5.71), turned to 90 degrees
- moved R6 3.86 mm to (43.2, 26.7)
- moved R5 3.81 mm to (45.7, 26.6)
- moved L2 1.80 mm to (69.8, 9.53), turned to 0 degrees
- moved R16 0.63 mm to (31.8, 21.6)
- moved L1 0.25 mm to (71.1, 18.0)
- moved R8 0.09 mm to (54.6, 13.8)
Connections:
- removed net N$15: L2.2, USB1.P1
- removed net OUT1: U6.7
- new net !VREG_EN: J6.1, U6.7
- new net ADC0: J6.2, U6.61
- new net N$13: F1.1, USB1.P1
- new net N$14: F1.2, L2.2
- net GND: now also J6.3
Routing:
- net ADC0: track 0.00 -> 29.2 mm, vias 0 -> 3
- net !VREG_EN: track 0.00 -> 28.9 mm, vias 0 -> 1
- net VIN: track 42.6 -> 38.8 mm
- net N$5: track 5.22 -> 8.92 mm
- net SW1: track 51.3 -> 54.5 mm
- net VUSB: track 21.5 -> 18.7 mm
- net UART_RX: track 29.1 -> 30.8 mm
- net UART_TX: track 28.6 -> 30.2 mm
- net RTC_EN: track 33.5 -> 34.4 mm
- net N$20: track 30.0 -> 29.3 mm
- net +5V: track 210.2 -> 209.6 mm
- added copper zone on layer 1, net N$13
- added copper zone on layer 1, net N$14
- removed copper zone on layer 1, net N$15
Other:
- board text added: "!VREG_EN"
- board text added: "ADC"
- board text added: "VREG CTRL"
